File: KiCad/Motion controller MiYR interface/Motion controller MiYR interface.kicad_pcb (KiCad board)
At the start: 4 copper layers, 78.5 x 196.3 mm, 87 parts, among them CN1 Conn_02x40_Odd_Even, CN2 Conn_02x40_Odd_Even, J1 10061913-111PLF, J2 10061913-111PLF, J3 10061913-111PLF, J4 10061913-111PLF, J5 Conn_01x02_Pin, U1 AP63201WU, U10 D1213A-04S-7, U11 D1213A-04S-7, U12 D1213A-04S-7, U13 D1213A-04S-7, U14 D1213A-04S-7, U15 D1213A-04S-7, U16 D1213A-04S-7, U17 D1213A-04S-7, U18 D1213A-04S-7, U19 D1213A-04S-7, U2 AOZ1360AIL, U20 D1213A-04S-7, U21 D1213A-04S-7, U22 D1213A-04S-7, U23 AOZ1360AIL, U24 AP63201WU, U25 AOZ1360AIL, U26 AP63201WU, U3 D1213A-04S-7, U30 D1213A-04S-7, U31 D1213A-04S-7, U32 D1213A-04S-7, U33 D1213A-04S-7, U4 D1213A-04S-7, U5 D1213A-04S-7, U6 D1213A-04S-7, U7 D1213A-04S-7, U8 D1213A-04S-7, U9 D1213A-04S-7

Commit message: 10ch encoder card
Parts:
- added REF**: OSHW-Logo2_14.6x12mm_SilkScreen, Symbol:OSHW-Logo2_14.6x12mm_SilkScreen, F.Cu at (200.0, 238.0)
- added REF**: OSHW-Logo2_14.6x12mm_SilkScreen, Symbol:OSHW-Logo2_14.6x12mm_SilkScreen, B.Cu at (144.0, 238.0)
Other:
- board size 78.5 x 196.3 mm -> 86 x 198 mm
- board text added: "+24"
- board text added: "GND"
- board text added: "SLOT A"
- board text added: "SLOT B"
- board text added: "SLOT C"
- board text added: "SLOT D"

Commit message: update controller boards
Parts:
- added REF**: MountingHole_3.2mm_M3_ISO14580_Pad_TopBottom, MountingHole:MountingHole_3.2mm_M3_ISO14580_Pad_TopBottom, F.Cu at (211.0, 157.0)
- added REF**: MountingHole_3.2mm_M3_ISO14580_Pad_TopBottom, MountingHole:MountingHole_3.2mm_M3_ISO14580_Pad_TopBottom, F.Cu at (211.0, 115.0)
- added REF**: MountingHole_3.2mm_M3_ISO14580_Pad_TopBottom, MountingHole:MountingHole_3.2mm_M3_ISO14580_Pad_TopBottom, F.Cu at (132.5, 55.0)
- added REF**: MountingHole_3.2mm_M3_ISO14580_Pad_TopBottom, MountingHole:MountingHole_3.2mm_M3_ISO14580_Pad_TopBottom, F.Cu at (132.5, 91.0)
- added REF**: EO silk 14mm, Library:EO silk 14mm, B.Cu at (202.0, 236.0)
- added REF**: MountingHole_3.2mm_M3_ISO14580_Pad_TopBottom, MountingHole:MountingHole_3.2mm_M3_ISO14580_Pad_TopBottom, F.Cu at (211.0, 74.0)
- added REF**: MountingHole_3.2mm_M3_ISO14580_Pad_TopBottom, MountingHole:MountingHole_3.2mm_M3_ISO14580_Pad_TopBottom, F.Cu at (211.0, 245.0)
- added REF**: MountingHole_3.2mm_M3_ISO14580_Pad_TopBottom, MountingHole:MountingHole_3.2mm_M3_ISO14580_Pad_TopBottom, F.Cu at (211.0, 201.0)
- added REF**: MountingHole_3.2mm_M3_ISO14580_Pad_TopBottom, MountingHole:MountingHole_3.2mm_M3_ISO14580_Pad_TopBottom, F.Cu at (132.5, 245.0)
- added REF**: MountingHole_3.2mm_M3_ISO14580_Pad_TopBottom, MountingHole:MountingHole_3.2mm_M3_ISO14580_Pad_TopBottom, F.Cu at (132.5, 201.0)
- added REF**: EO silk 14mm, Library:EO silk 14mm, F.Cu at (140.2, 237.2)
- added REF**: MountingHole_3.2mm_M3_ISO14580_Pad_TopBottom, MountingHole:MountingHole_3.2mm_M3_ISO14580_Pad_TopBottom, F.Cu at (132.5, 157.0)
- C6: footprint Capacitor_SMD:C_0603_1608Metric -> Capacitor_SMD:C_1206_3216Metric
