File: KiCad/Motion controller MiYR interface/Motion controller MiYR interface.kicad_sch (KiCad schematic)
At the start: 136 parts, among them CN1 Conn_02x40_Odd_Even, CN2 Conn_02x40_Odd_Even, J1 10061913-111PLF, J2 10061913-111PLF, J3 10061913-111PLF, J4 10061913-111PLF, J5 Conn_01x02_Pin, U1 AP63201WU, U10 D1213A-04S-7, U11 D1213A-04S-7, U12 D1213A-04S-7, U13 D1213A-04S-7, U14 D1213A-04S-7, U15 D1213A-04S-7, U16 D1213A-04S-7, U17 D1213A-04S-7, U18 D1213A-04S-7, U19 D1213A-04S-7, U2 AOZ1360AIL, U20 D1213A-04S-7, U21 D1213A-04S-7, U22 D1213A-04S-7, U23 AOZ1360AIL, U24 AP63201WU, U25 AOZ1360AIL, U26 AP63201WU, U3 D1213A-04S-7, U30 D1213A-04S-7, U31 D1213A-04S-7, U32 D1213A-04S-7, U33 D1213A-04S-7, U34 74HC165, U35 74HC595, U36 LM324, U37 LM324, U4 D1213A-04S-7, U5 D1213A-04S-7, U6 D1213A-04S-7, U7 D1213A-04S-7, U8 D1213A-04S-7, U9 D1213A-04S-7

Commit message: update controller boards
Parts:
- C6: footprint Capacitor_SMD:C_0603_1608Metric -> Capacitor_SMD:C_1206_3216Metric
Other:
- note added: "RGB led"
